File: V3.1-H1/brake-estop.kicad_sch (KiCad schematic)
At the start: 31 parts

Commit message: Merge the E-stop relays and rename ESTOP_JET to ESTOP_REMOTE
The four E-stop relays become ESTOP_COM_RELAY1 and ESTOP_COM_RELAY2.
Each keeps the coil of its BOMAG relay and takes the CAT contacts on
its spare pole. The support parts follow the new names and the second
series diode is removed.

Co-Authored-By: Claude Fable 5.1 <noreply@anthropic.com>
Parts:
- removed D_ESTOPJET_SER2, D_KESTOPCAT1, D_KESTOPCAT2: D, 1N4148WS:SOD-323_L1.8-W1.3-LS2.5-RD, symbol Device:D
- removed ESTOPCAT1-Relay-LED1, ESTOPCAT2-Relay-LED1: Green, LED_SMD:LED_0805_2012Metric, symbol Device:LED
- removed ESTOPCAT1-Relay-RES1, ESTOPCAT2-Relay-RES1: 2.2k, Resistor_SMD:R_0805_2012Metric, symbol Device:R
- removed K_ESTOP_CAT1, K_ESTOP_CAT2: Relay_DPDT, Relay_THT:Relay_DPDT_Omron_G6A, symbol Relay:Relay_DPDT
- renumbered D_KESTOPBOMAG1 to D_ESTOPCOM1, D_KESTOPBOMAG2 to D_ESTOPCOM2, D_ESTOPJET_SER1 to D_ESTOPREMOTE_SER1, ESTOPBOMAG1-Relay-LED1 to ESTOPCOM1-Relay-LED1, ESTOPBOMAG1-Relay-RES1 to ESTOPCOM1-Relay-RES1, ESTOPBOMAG2-Relay-LED1 to ESTOPCOM2-Relay-LED1, ESTOPBOMAG2-Relay-RES1 to ESTOPCOM2-Relay-RES1, K_ESTOP_BOMAG1 to ESTOP_COM_RELAY1, K_ESTOP_BOMAG2 to ESTOP_COM_RELAY2
Connections:
- net ESTOP_CAT_RELAY: now also ESTOP_COM_RELAY1.14, ESTOP_COM_RELAY2.11
- net ESTOP_ECU_NF: now also ESTOP_COM_RELAY2.12
- net ESTOP_ECU_NG: now also ESTOP_COM_RELAY1.12, ESTOP_COM_RELAY2.14
- net ESTOP_JOY_NG: now also ESTOP_COM_RELAY1.11
- net ESTOP_JET renamed ESTOP_REMOTE
- no-connect marks 17 -> 5
Other:
- note added: "ESTOP COM RELAY1"
- note added: "ESTOP COM RELAY2"
- note removed: "ESTOP BOMAG1 RELAY"
- note removed: "ESTOP BOMAG2 RELAY"
- note removed: "ESTOP CAT1 RELAY"
- note removed: "ESTOP CAT2 RELAY"
