File: V3.1-H1/CREWLINE-PRIM-PCB-001.kicad_pcb (KiCad board)
At the start: 4 copper layers, 101 x 132 mm, 78 parts, among them J1 BATTERY, J2 CHARGE SHIELD HEADER, J3 DIO, J4 PWR INPUTS, J5 CAN CABLES, J6 SEAT_CONNECTOR, J7 BRAKE INPUTS, J8 SAFETY_CONNECTOR, J9 Conn_02x06_Counter_Clockwise, Q1 IRF4905STRL

Commit message: Grow the board and route the new relay and connector circuits
Widen the board by 56.5 mm so J5, J7 and J10 fit on the bottom edge.
Move J8, J6, the test point column and the right-hand mounting holes
with the edge. Place seven DPDT relays in one row above the connectors
with their diodes, LEDs and resistors, and add the five new test points.

Route all new connections on the outer layers with a grid router that
keeps the clearance rules, the mounting hole washer areas and a 2 mm
edge margin. The CAN pair runs side by side. DRC reports no errors,
no warnings and no unconnected items.

Trim the XT60 silkscreen at the board edge in the project library and
move the J4 reference clear of its test point.

Co-Authored-By: Claude Fable 5.1 <noreply@anthropic.com>
Parts:
- added BRKCAT1-Relay-LED1: Green, LED_SMD:LED_0805_2012Metric, F.Cu at (127.2, 137.0)
- added BRKCAT1-Relay-RES1: 2.2k, Resistor_SMD:R_0805_2012Metric, F.Cu at (123.2, 137.0)
- added BRKCAT2-Relay-LED1: Green, LED_SMD:LED_0805_2012Metric, F.Cu at (140.7, 137.0)
- added BRKCAT2-Relay-RES1: 2.2k, Resistor_SMD:R_0805_2012Metric, F.Cu at (136.7, 137.0)
- added BRK_ECU_NF_TP1: TestPoint, TestPoint_Black:TEST-TH_BD2.54-P1.4_BLACK, F.Cu at (188.0, 151.0)
- added BRK_ECU_NG_TP1: TestPoint, TestPoint_Black:TEST-TH_BD2.54-P1.4_BLACK, F.Cu at (188.0, 147.0)
- added D_BRAKEJET_SER1: D, 1N4148WS:SOD-323_L1.8-W1.3-LS2.5-RD, F.Cu at (138.8, 134.0)
- added D_ESTOPCOM1: D, 1N4148WS:SOD-323_L1.8-W1.3-LS2.5-RD, F.Cu at (155.8, 140.0)
- added D_ESTOPCOM2: D, 1N4148WS:SOD-323_L1.8-W1.3-LS2.5-RD, F.Cu at (169.3, 140.0)
- added D_ESTOPREMOTE_SER1: D, 1N4148WS:SOD-323_L1.8-W1.3-LS2.5-RD, F.Cu at (169.3, 134.0)
- added D_KBRAKECAT1: D, 1N4148WS:SOD-323_L1.8-W1.3-LS2.5-RD, F.Cu at (125.3, 140.0)
- added D_KBRAKECAT2: D, 1N4148WS:SOD-323_L1.8-W1.3-LS2.5-RD, F.Cu at (138.8, 140.0)
- added ESTOPCOM1-Relay-LED1: Green, LED_SMD:LED_0805_2012Metric, F.Cu at (157.7, 137.0)
- added ESTOPCOM1-Relay-RES1: 2.2k, Resistor_SMD:R_0805_2012Metric, F.Cu at (153.7, 137.0)
- added ESTOPCOM2-Relay-LED1: Green, LED_SMD:LED_0805_2012Metric, F.Cu at (171.2, 137.0)
- added ESTOPCOM2-Relay-RES1: 2.2k, Resistor_SMD:R_0805_2012Metric, F.Cu at (167.2, 137.0)
- added ESTOP_COM_RELAY1: Relay_DPDT, Relay_THT:Relay_DPDT_Omron_G6A, F.Cu at (152.0, 143.2)
- added ESTOP_COM_RELAY2: Relay_DPDT, Relay_THT:Relay_DPDT_Omron_G6A, F.Cu at (165.5, 143.2)
- added ESTP_ECU_NF_TP1: TestPoint, TestPoint_Black:TEST-TH_BD2.54-P1.4_BLACK, F.Cu at (188.0, 163.0)
- added ESTP_ECU_NG_TP1: TestPoint, TestPoint_Black:TEST-TH_BD2.54-P1.4_BLACK, F.Cu at (188.0, 159.0)
- added ESTP_ECU_TP1: TestPoint, TestPoint_Black:TEST-TH_BD2.54-P1.4_BLACK, F.Cu at (188.0, 155.0)
- added J10: ESTOP INPUTS, V31_H1:MCV_1.5_7_5.08_Pad2.6, F.Cu at (161.2, 173.0)
- added K_BRAKE_CAT1: Relay_DPDT, Relay_THT:Relay_DPDT_Omron_G6A, F.Cu at (121.5, 143.2)
- added K_BRAKE_CAT2: Relay_DPDT, Relay_THT:Relay_DPDT_Omron_G6A, F.Cu at (135.0, 143.2)
- J7: footprint V31_H1:MCV_1.5_4_5.08_Pad2.6 -> V31_H1:MCV_1.5_7_5.08_Pad2.6
- moved BRK_ECU_TP1 56.6 mm to (202.1, 164.5)
- moved CAN1L_TP1 56.5 mm to (202.1, 161.0)
- moved CAN1H_TP1 56.5 mm to (202.1, 157.5)
- moved KIT_TP1 56.5 mm to (202.0, 154.0)
- moved 12V_GATE_TP1 56.5 mm to (202.0, 150.5)
- moved J6 56.5 mm to (204.0, 135.0)
- moved J8 56.5 mm to (199.0, 125.7)
- moved MODE_TP1 56.5 mm to (202.0, 147.0)
- moved REF** 56.5 mm to (201.5, 173.5)
- moved REF** 56.5 mm to (200.5, 56.5)
- moved D_KBRAKE1 23.5 mm to (111.8, 140.0)
- moved D_KECUCAN1 21.7 mm to (80.8, 140.0)
- moved D_KJOYCAN1 21.2 mm to (94.3, 140.0)
- moved Joy-Relay-LED1 8.32 mm to (96.2, 137.0)
- moved Joy-Relay-RES1 8.20 mm to (92.2, 137.0)
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- renumbered K_BRAKE1 to K_BRAKE_BOMAG1
Connections:
- J7 pad 4: unconnected-(J7-Pin_4-Pad4) -> BRAKE_JOY_NG
Routing:
- net BRAKE_ECU_NF: track 0.00 -> 102.9 mm
- net BRAKE_ECU: track 43.6 -> 125.4 mm
- net JET1_CANH: track 83.6 -> 159.8 mm
- net BRAKE_ECU_NG: track 0.00 -> 76.0 mm
- net +12V_KIT: track 207.4 -> 135.6 mm, vias 0 -> 10
- net JET1_CANL: track 77.7 -> 149.5 mm, vias 2 -> 4
- net ESTOP_ECU: track 0.00 -> 70.4 mm, vias 0 -> 2
- net MODE_SEL_DRV: track 168.9 -> 239.2 mm, vias 0 -> 1
- net ESTOP_ECU_NF: track 0.00 -> 61.9 mm
- net BRAKE_JET: track 12.8 -> 72.8 mm, vias 0 -> 1
- net ESTOP_REMOTE: track 0.00 -> 58.1 mm, vias 0 -> 1
- net ESTOP_ECU_NG: track 0.00 -> 57.6 mm
- net ARMED_HOT: track 63.6 -> 119.9 mm
- net +12V_GATED: track 165.2 -> 220.7 mm, vias 0 -> 1
- net ESTOP_JOY_NG: track 0.00 -> 52.9 mm
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Other:
- board size 101 x 132 mm -> 157.5 x 132 mm
- board text added: "BRK NF"
- board text added: "BRK NG"
- board text added: "ES NF"
- board text added: "ES NG"
- board text added: "ESTOP"
