File: new/brake-estop.kicad_sch (KiCad schematic)
At the start: 22 parts

Commit message: Apply the routine findings of the independent review
Via sizes now follow the net class, and +12V_GATED and +12V_KIT are
re-routed with them. Relay references sit below the relay bodies with
a 0.15 mm stroke. The mounting holes are H1 to H4, board-only, on a
rectangular pattern. Diodes carry the value 1N4148WS. The README
records the re-routed nets, the disabled checks and the open items.
Derived files regenerated.

Co-Authored-By: Claude Fable 5.1 <noreply@anthropic.com>
Parts:
- D_BRAKEJET_SER1, D_ESTOPCOM1, D_ESTOPCOM2, D_ESTOPREMOTE_SER1, D_KBRAKE1, D_KBRAKECAT1, D_KBRAKECAT2: value D -> 1N4148WS
Changed lines of the file:
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@@
 			)
 		)
-		(property "Value" "D"
+		(property "Value" "1N4148WS"
 			(at 45.72 22.86 0)
 			(show_name no)
@@
 			)
 		)
-		(property "Value" "D"
+		(property "Value" "1N4148WS"
 			(at 106.68 22.86 0)
 			(show_name no)
@@
 			)
 		)
-		(property "Value" "D"
+		(property "Value" "1N4148WS"
 			(at 116.84 37.465 0)
 			(hide yes)
@@
 			)
 		)
-		(property "Value" "D"
+		(property "Value" "1N4148WS"
 			(at 170.18 22.86 0)
 			(show_name no)
@@
 			)
 		)
-		(property "Value" "D"
+		(property "Value" "1N4148WS"
 			(at 45.72 74.93 0)
 			(show_name no)
@@
 			)
 		)
-		(property "Value" "D"
+		(property "Value" "1N4148WS"
 			(at 106.68 74.93 0)
 			(show_name no)
@@
 			)
 		)
-		(property "Value" "D"
+		(property "Value" "1N4148WS"
 			(at 116.84 89.535 0)
 			(hide yes)
