File: new/CREWLINE-PRIM-PCB-001.kicad_pcb (KiCad board)
At the start: 4 copper layers, 157.5 x 132 mm, 102 parts, among them J1 BATTERY, J10 ESTOP INPUTS, J2 CHARGE SHIELD HEADER, J3 DIO, J4 PWR INPUTS, J5 CAN CABLES, J6 SEAT_CONNECTOR, J7 BRAKE INPUTS, J8 SAFETY_CONNECTOR, J9 Conn_02x06_Counter_Clockwise, Q1 IRF4905STRL

Commit message: Apply the routine findings of the independent review
Via sizes now follow the net class, and +12V_GATED and +12V_KIT are
re-routed with them. Relay references sit below the relay bodies with
a 0.15 mm stroke. The mounting holes are H1 to H4, board-only, on a
rectangular pattern. Diodes carry the value 1N4148WS. The README
records the re-routed nets, the disabled checks and the open items.
Derived files regenerated.

Co-Authored-By: Claude Fable 5.1 <noreply@anthropic.com>
Parts:
- D1, D2, D_BRAKEJET_SER1, D_ESTOPCOM1, D_ESTOPCOM2, D_ESTOPREMOTE_SER1, D_KBRAKE1, D_KBRAKECAT1, D_KBRAKECAT2, D_KECUCAN1, D_KJOYCAN1, D_KSTEER1: value D -> 1N4148WS
- moved H2 1.80 mm to (201.5, 58.0)
- moved H4 0.50 mm to (201.5, 173.0)
- renumbered REF** to H1, REF** to H2, REF** to H3, REF** to H4
Other:
- board text added: "ES ECU"
- board text removed: "ESTOP"

Commit message: Move the CAN test points beside J5 and record the review outcomes
CAN1H_TP1 and CAN1L_TP1 now sit above J5 pins 6 to 9 so their stubs on
the bus are short, and the pair is routed together. Relay references
stand in the gap beside each body. The README records the BRAKE_JET
supply limit and the open questions for the original designer.

Co-Authored-By: Claude Fable 5.1 <noreply@anthropic.com>
Parts:
- moved CAN1H_TP1 96.3 mm to (106.0, 165.0)
- moved CAN1L_TP1 91.6 mm to (110.5, 165.0)
- moved BRK_ECU_TP1 7.00 mm to (202.1, 157.5)
Routing:
- net JET1_CANH: track 159.8 -> 37.2 mm, vias 1 -> 0
- net JET1_CANL: track 149.5 -> 33.6 mm, vias 4 -> 1
- net BRAKE_ECU: track 125.4 -> 132.4 mm

Commit message: Swap the signal connectors to Molex Micro-Fit, audit the BOM, shrink the board
J3, J5, J6, J7 and J10 are Molex Micro-Fit 3.0 single-row through-hole
headers. J8, J2 and all test points are removed; the arming loop moves to
J3 and J6 becomes the seat sensor connector. The red LEDs use the
standard symbol so pad 1 is the cathode. D1 is turned round and
R_ARMED_PD1 removed. Every part number was checked against the JLCPCB
library and corrected; J4 and the fuse holders are marked customer
fitted. The board shrinks to 136 x 132 mm with the mounting holes on a
120 x 115 mm rectangle. Footprint fields are synced so the parity check
is clean. Derived files regenerated and README rewritten.

Co-Authored-By: Claude Fable 5.1 <noreply@anthropic.com>
Parts:
- removed 12V_GATE_TP1, BATT_TP1, CONV_TP1, DIO_TP1, JET_TP3, KIT_TP1, LED_TP1, STAR_TP1, STR_TP1: TestPoint, TestPoint_Red:TEST-TH_BD2.54-P1.4_RED
- removed ARM_TP1, BATT_GND_TP1, BRK_ECU_NF_TP1, BRK_ECU_NG_TP1, BRK_ECU_TP1, CAN1H_TP1, CAN1L_TP1, ESTP_ECU_NF_TP1, ESTP_ECU_NG_TP1, ESTP_ECU_TP1, MODE_TP1: TestPoint, TestPoint_Black:TEST-TH_BD2.54-P1.4_BLACK
- removed J2: CHARGE SHIELD HEADER, Connector_PinSocket_2.54mm:PinSocket_2x04_P2.54mm_Vertical
- removed J8: SAFETY_CONNECTOR, V31_H1:MCV_1.5_5_5.08_Pad2.6
- removed K_BRAKE_BOMAG1: Relay_DPDT, Relay_THT:Relay_DPDT_Omron_G6A
- removed R_ARMED_PD1: 10k, Resistor_SMD:R_0805_2012Metric
- added K_BRAKE_SEAT_BOMAG1: G6A-274P-ST-US-DC12, Relay_THT:Relay_DPDT_Omron_G6A, F.Cu at (103.2, 145.0)
- ESTOP_COM_RELAY1, ESTOP_COM_RELAY2, K_BRAKE_CAT1, K_BRAKE_CAT2, K_ECUCAN1, K_JOYCAN1: value Relay_DPDT -> G6A-274P-ST-US-DC12
- J10, J7: footprint V31_H1:MCV_1.5_7_5.08_Pad2.6 -> Connector_Molex:Molex_Micro-Fit_3.0_43650-0715_1x07_P3.00mm_Vertical
- J3: value DIO -> MODE_SEL/PWR GATE; footprint V31_H1:MCV_1.5_5_5.08_Pad2.6 -> Connector_Molex:Molex_Micro-Fit_3.0_43650-0515_1x05_P3.00mm_Vertical
- J5: footprint V31_H1:MCV_1.5_10_5.08_Pad2.6 -> Connector_Molex:Molex_Micro-Fit_3.0_43650-1015_1x10_P3.00mm_Vertical
- J6: value SEAT_CONNECTOR -> SEAT SENSOR; footprint WAGO_2604:WAGO_2604-1102 -> Connector_Molex:Molex_Micro-Fit_3.0_43650-0315_1x03_P3.00mm_Vertical
- POWER1: value K_GATE -> SLA-12VDC-SL-A
- moved J6 143.6 mm to (62.3, 158.3)
- moved H2 21.5 mm to (180.0, 58.0)
- moved H4 21.5 mm to (180.0, 173.0)
- moved D_ESTOPREMOTE_SER1 19.5 mm to (153.9, 145.9), turned to -90 degrees
- moved J7 18.0 mm to (105.0, 173.0)
- moved J10 17.2 mm to (144.0, 173.0)
- moved JOY_TERM_R1 13.5 mm to (89.1, 167.1)
- moved STEER_TERM_R1 13.5 mm to (89.0, 165.1)
- moved D_BRAKEJET_SER1 12.7 mm to (128.8, 141.9), turned to 180 degrees
- moved ESTOPCOM1-Relay-RES1 11.4 mm to (142.5, 138.8)
- moved ESTOP_COM_RELAY1 10.3 mm to (141.8, 145.0)
- moved ESTOPCOM1-Relay-LED1 9.40 mm to (148.5, 138.8)
- moved D_ESTOPCOM1 8.54 mm to (147.5, 141.8)
- moved ESTOPCOM2-Relay-RES1 7.50 mm to (159.9, 138.7)
- moved ESTOP_COM_RELAY2 7.10 mm to (158.6, 145.0)
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Connections:
- CONV_LED1 pad 1: CONV_PWR_P -> Net-(CONV_LED1-K)
- CONV_LED1 pad 2: Net-(CONV_LED1-C) -> CONV_PWR_P
- CONV_RES1 pad 1: Net-(CONV_LED1-C) -> Net-(CONV_LED1-K)
- D1 pad 1: GND -> ARMED_HOT
- D1 pad 2: ARMED_HOT -> GND
- DIO_LED1 pad 1: JET_DIO_PWR_P -> Net-(DIO_LED1-K)
- DIO_LED1 pad 2: Net-(DIO_LED1-C) -> JET_DIO_PWR_P
- DIO_RES1 pad 1: Net-(DIO_LED1-C) -> Net-(DIO_LED1-K)
- J10 pad 1: ESTOP_REMOTE -> ESTOP_JOY_NG
- J10 pad 4: ESTOP_JOY_NG -> ESTOP_REMOTE
- J10 pad 6: ESTOP_ECU_NG -> ESTOP_ECU_NF
- J10 pad 7: ESTOP_ECU_NF -> ESTOP_ECU_NG
- J3 pad 2: /FAULT -> +12V_GATED
- J3 pad 3: VEHICLE_ON -> Net-(J3-Pin_3)
- J3 pad 4: /CHRG -> Net-(J3-Pin_3)
- J3 pad 5: VBAT_SENSE -> ARMED_HOT
- J6 pad 1: unconnected-(J6-Pin_1-Pad1) -> ECU_SEAT
- J6 pad 2: MODE_SEL_DRV -> SEAT
- J7 pad 4: BRAKE_JOY_NG -> BRAKE_JOY_NF
- J7 pad 5: BRAKE_JOY_NF -> BRAKE_JOY_NG
- J7 pad 6: BRAKE_ECU_NG -> BRAKE_ECU_NF
- J7 pad 7: BRAKE_ECU_NF -> BRAKE_ECU_NG
- JET_LED1 pad 1: JETSON_PWR_P -> Net-(JET_LED1-K)
- JET_LED1 pad 2: Net-(JET_LED1-C) -> JETSON_PWR_P
- JET_RES1 pad 1: Net-(JET_LED1-C) -> Net-(JET_LED1-K)
- LED_LED1 pad 1: LED_PWR_P -> Net-(LED_LED1-K)
- LED_LED1 pad 2: Net-(LED_LED1-C) -> LED_PWR_P
- LED_RES1 pad 1: Net-(LED_LED1-C) -> Net-(LED_LED1-K)
- PWR_LIGHT1 pad 1: +12V_KIT -> Net-(D2-A)
- PWR_LIGHT1 pad 2: Net-(D2-A) -> +12V_KIT
- STR_LED1 pad 1: STEER_PWR_P -> Net-(STR_LED1-K)
- STR_LED1 pad 2: Net-(STR_LED1-C) -> STEER_PWR_P
- STR_RES1 pad 1: Net-(STR_LED1-C) -> Net-(STR_LED1-K)
Routing:
- net MODE_SEL_DRV: track 239.2 -> 122.2 mm, vias 1 -> 0
- net BRAKE_ECU: track 132.4 -> 22.4 mm
- net BRAKE_ECU_NF: track 102.9 -> 24.1 mm
- net +12V_GATED: track 220.7 -> 147.3 mm, vias 1 -> 0
- net SEAT: track 0.00 -> 55.8 mm
- net +12V_KIT: track 135.6 -> 186.1 mm, vias 10 -> 0
- net BRAKE_ECU_NG: track 76.0 -> 26.0 mm
- net ESTOP_ECU: track 70.4 -> 21.3 mm, vias 2 -> 0
- net ECU_SEAT: track 0.00 -> 43.1 mm
- net ESTOP_ECU_NF: track 61.9 -> 19.7 mm
- net VEHICLE_ON: track 33.3 -> 0.00 mm
- net ESTOP_REMOTE: track 58.1 -> 26.3 mm, vias 1 -> 0
- net ESTOP_JOY_NG: track 52.9 -> 21.3 mm
- net BRAKE_JET: track 72.8 -> 42.7 mm
- net /FAULT: track 23.7 -> 0.00 mm
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Other:
- board size 157.5 x 132 mm -> 136 x 132 mm
- board text removed: "2"
- board text removed: "4"
- board text removed: "6"
- board text removed: "8"
- board text removed: "BRK NF"
- board text removed: "BRK NG"
- board text removed: "CAN1H"
- board text removed: "CAN1L"
- board text removed: "ECU BRAKE"
- board text removed: "ECU_CANL"
- board text removed: "ES ECU"
- board text removed: "ES NF"
- board text removed: "ES NG"
