File: new/_restore_backup_2026-09-30T12-59-34-863/brake-estop.kicad_sch (KiCad schematic)
At the start: 22 parts

Commit message: Swap the signal connectors to Molex Micro-Fit, audit the BOM, shrink the board
J3, J5, J6, J7 and J10 are Molex Micro-Fit 3.0 single-row through-hole
headers. J8, J2 and all test points are removed; the arming loop moves to
J3 and J6 becomes the seat sensor connector. The red LEDs use the
standard symbol so pad 1 is the cathode. D1 is turned round and
R_ARMED_PD1 removed. Every part number was checked against the JLCPCB
library and corrected; J4 and the fuse holders are marked customer
fitted. The board shrinks to 136 x 132 mm with the mounting holes on a
120 x 115 mm rectangle. Footprint fields are synced so the parity check
is clean. Derived files regenerated and README rewritten.

Co-Authored-By: Claude Fable 5.1 <noreply@anthropic.com>
Parts:
- BRK-Relay-LED1, BRKCAT1-Relay-LED1, BRKCAT2-Relay-LED1, ESTOPCOM1-Relay-LED1, ESTOPCOM2-Relay-LED1: LCSC Part C2297 -> C72043; MPN KT-0805G -> (none); Manufacturer KENTO -> (none)
- BRK-Relay-RES1, BRKCAT1-Relay-RES1, BRKCAT2-Relay-RES1, ESTOPCOM1-Relay-RES1, ESTOPCOM2-Relay-RES1: LCSC Part C17520 -> C25879
- D_BRAKEJET_SER1, D_ESTOPCOM1, D_ESTOPCOM2, D_ESTOPREMOTE_SER1, D_KBRAKE1, D_KBRAKECAT1, D_KBRAKECAT2: LCSC Part C2128 -> C81598; MPN 1N4148WS -> (none)
- ESTOP_COM_RELAY1, ESTOP_COM_RELAY2, K_BRAKE_CAT1, K_BRAKE_CAT2: value G6A-274P-ST-US-DC12 -> Relay_DPDT; LCSC Part C129439 -> C45404; MPN G6A-274P-ST-US-DC12 -> (none); Manufacturer Omron -> (none)
- K_BRAKE_BOMAG1: renamed from K_BRAKE_SEAT_BOMAG1; value G6A-274P-ST-US-DC12 -> Relay_DPDT; LCSC Part C129439 -> C45404; MPN G6A-274P-ST-US-DC12 -> (none); Manufacturer Omron -> (none)
Connections:
- net GND: no longer K_BRAKE_BOMAG1.14
- net ECU_SEAT: no longer names the net of K_BRAKE_BOMAG1.12
- net SEAT: no longer names the net of K_BRAKE_BOMAG1.11
- no-connect marks 2 -> 5
