File: new/_restore_backup_2026-10-01T12-37-35-978/CREWLINE-PRIM-PCB-001.kicad_sch (KiCad schematic)
At the start: 53 parts, among them J1 BATTERY, J10 ESTOP INPUTS, J3 MODE_SEL/PWR GATE, J4 PWR INPUTS, J5 CAN CABLES, J6 SEAT SENSOR, J7 BRAKE INPUTS, J9 Conn_02x06_Counter_Clockwise, Q1 IRF4905STRL

Commit message: Swap the signal connectors to Molex Micro-Fit, audit the BOM, shrink the board
J3, J5, J6, J7 and J10 are Molex Micro-Fit 3.0 single-row through-hole
headers. J8, J2 and all test points are removed; the arming loop moves to
J3 and J6 becomes the seat sensor connector. The red LEDs use the
standard symbol so pad 1 is the cathode. D1 is turned round and
R_ARMED_PD1 removed. Every part number was checked against the JLCPCB
library and corrected; J4 and the fuse holders are marked customer
fitted. The board shrinks to 136 x 132 mm with the mounting holes on a
120 x 115 mm rectangle. Footprint fields are synced so the parity check
is clean. Derived files regenerated and README rewritten.

Co-Authored-By: Claude Fable 5.1 <noreply@anthropic.com>
Parts:
- C1: LCSC Part C338185 -> C44650
- CONV_LED1, DIO_LED1, JET_LED1, LED_LED1, PWR_LIGHT1, STR_LED1: symbol Device:LED -> V31_H1:LED_Red_0805_A1; LCSC Part C2295 -> (none); MPN KT-0805R -> (none); Manufacturer KENTO -> (none)
- CONV_RES1, DIO_RES1, ECU-Relay-RES1, JET_RES1, Joy-Relay-RES1, LED_RES1, STR-Relay-RES1, STR_RES1: LCSC Part C17520 -> C25879
- C_STEER1: LCSC Part C1669326 -> C44897
- D1, D2, D_KECUCAN1, D_KJOYCAN1, D_KSTEER1: LCSC Part C2128 -> C81598; MPN 1N4148WS -> (none)
- ECU-Relay-LED4, Joy-Relay-LED1, STR-Relay-LED1: LCSC Part C2297 -> C72043; MPN KT-0805G -> (none); Manufacturer KENTO -> (none)
- F_CONV1, F_DIO1, F_JET1, F_LED1, F_STEER1: Assembly Customer fitted -> (none); LCSC Part (none) -> DNP; MPN 3568 -> (none); Manufacturer Keystone -> (none)
- F_MAIN1: Assembly Customer fitted -> (none); LCSC Part (none) -> DNP; MPN 3568 -> 0297030.U; Manufacturer Keystone -> (none)
- J10, J7: footprint Connector_Molex:Molex_Micro-Fit_3.0_43650-0715_1x07_P3.00mm_Vertical -> V31_H1:MCV_1.5_7_5.08_Pad2.6; LCSC Part C17199797 -> (none); MPN 43650-0715 -> 1836341; Manufacturer Molex -> Phoenix Contact; Mating plug 43645-0700 -> 1836121
- J3: footprint Connector_Molex:Molex_Micro-Fit_3.0_43650-0515_1x05_P3.00mm_Vertical -> V31_H1:MCV_1.5_5_5.08_Pad2.6; LCSC Part C505230 -> (none); MPN 43650-0515 -> 1836325; Manufacturer Molex -> Phoenix Contact; Mating plug 43645-0500 -> 1836105
- J4: Assembly Customer fitted -> (none); LCSC Part (none) -> DNP; MPN 1715802 -> (none); Manufacturer Phoenix Contact -> (none)
- J5: footprint Connector_Molex:Molex_Micro-Fit_3.0_43650-1015_1x10_P3.00mm_Vertical -> V31_H1:MCV_1.5_10_5.08_Pad2.6; LCSC Part C17337723 -> (none); MPN 43650-1015 -> 1836370; Manufacturer Molex -> Phoenix Contact; Mating plug 43645-1000 -> 1836150
- J6: footprint Connector_Molex:Molex_Micro-Fit_3.0_43650-0315_1x03_P3.00mm_Vertical -> V31_H1:MCV_1.5_2_5.08_Pad2.6; symbol Connector:Conn_01x03_Socket -> Connector:Conn_01x02_Socket; LCSC Part C293546 -> (none); MPN 43650-0315 -> 1836299; Manufacturer Molex -> Phoenix Contact; Mating plug 43645-0300 -> 1836079
- K_ECUCAN1, K_JOYCAN1: value G6A-274P-ST-US-DC12 -> Relay_DPDT; LCSC Part C129439 -> C45404; MPN G6A-274P-ST-US-DC12 -> (none); Manufacturer Omron -> (none)
- POWER1: value SLA-12VDC-SL-A -> K_GATE
- Q_MODE1: LCSC Part C155257 -> C700958; MPN DMN3404L-7 -> (none); Manufacturer Diodes Incorporated -> (none)
- R_ARMED1: LCSC Part C4382 -> C17475
- R_MODE_GATE1: LCSC Part C17408 -> C17561
- TVS1: LCSC Part C78416 -> C13616
Connections:
- net +12V_KIT: now also PWR_LIGHT1.1 (A); no longer PWR_LIGHT1.2 (A)
- net CONV_PWR_P: now also CONV_LED1.1 (A); no longer CONV_LED1.2 (A)
- net JETSON_PWR_P: now also JET_LED1.1 (A); no longer JET_LED1.2 (A)
- net JET_DIO_PWR_P: now also DIO_LED1.1 (A); no longer DIO_LED1.2 (A)
- net LED_PWR_P: now also LED_LED1.1 (A); no longer LED_LED1.2 (A)
- net STEER_PWR_P: now also STR_LED1.1 (A); no longer STR_LED1.2 (A)
- net at DIO_RES1.1: now also DIO_LED1.2 (C); no longer DIO_LED1.1 (K)
- net at STR_RES1.1: now also STR_LED1.2 (C); no longer STR_LED1.1 (K)
- net at D2.2 (A), R_ARMED1.1: now also PWR_LIGHT1.2 (C); no longer PWR_LIGHT1.1 (K)
- net at LED_RES1.1: now also LED_LED1.2 (C); no longer LED_LED1.1 (K)
- net at CONV_RES1.1: now also CONV_LED1.2 (C); no longer CONV_LED1.1 (K)
- net at JET_RES1.1: now also JET_LED1.2 (C); no longer JET_LED1.1 (K)
- no-connect marks 5 -> 4
